Commit message: Add files via upload

File: robot_model/PIPPA.urdf (robot description, URDF)
Before this commit: robot PIPPA, 19 links, 18 joints
Links:
- link Bottom_straight_link: geometry collision mesh filename=../Cylinder.stl scale=1.00000 1.00000 0.83333; visual mesh filename=../Cylinder.stl scale=1.00000 1.00000 0.83333
