Commit message: Update PIPPA.urdf

File: Robot/PIPPA/PIPPA.urdf (robot description, URDF)
Before this commit: robot PIPPA, 19 links, 18 joints
Links:
- link Bottom_straight_link: geometry collision mesh filename=Robot/PIPPA/Cylinder.stl scale=1.00000 1.00000 0.83333; visual mesh filename=Robot/PIPPA/Cylinder.stl scale=1.00000 1.00000 0.83333

Commit message: Update and rename PIPPA_deformable.urdf to PIPPA.urdf

File: Robot/PIPPA/PIPPA.urdf (robot description, URDF)
Before this commit: robot PIPPA, 19 links, 18 joints
Links:
- link Bottom_Link_1: mass 8.60000 -> 0.0
- link Bottom_Link_2: mass 8.60000 -> 0.0
- link Bottom_Link_3: mass 8.60000 -> 0.0
- link Colonna_Link_1: mass 0.05690 -> 8.6
- link Colonna_Link_2: mass 0.05690 -> 8.6
- link Colonna_Link_3: mass 0.05690 -> 8.6
- link Cover_Link1: mass 15.42300 -> 0.78
- link Cover_Link_2: mass 15.42300 -> 0.78
- link Cover_Link_3: mass 15.42300 -> 0.78
- link Gamba_Link_1: mass 0.78000 -> 1.6145
- link Gamba_Link_2: mass 0.78000 -> 1.6145
- link Gamba_Link_3: mass 0.78000 -> 1.6145
- link Top_Link_1: mass None -> 15.423
- link Top_Link_2: mass None -> 15.423
- link Top_Link_3: mass None -> 15.423

Commit message: Update PIPPA.urdf

File: Robot/PIPPA/PIPPA.urdf (robot description, URDF)
Before this commit: robot PIPPA, 19 links, 18 joints
Joints:
- added joint base_to_ground: type floating, parent world, child Bottom_straight_link

Commit message: Update PIPPA.urdf

File: Robot/PIPPA/PIPPA.urdf (robot description, URDF)
Before this commit: robot PIPPA, 19 links, 19 joints
Joints:
- removed joint base_to_ground

Commit message: Add files via upload

File: Robot/PIPPA/PIPPA.urdf (robot description, URDF)
Before this commit: robot PIPPA, 19 links, 18 joints
Links:
- added link Bottom_core, mass 0; collision mesh filename=Robot/PIPPA/Cylinder.033.stl scale=1.000 1.000 0.833; visual mesh filename=Robot/PIPPA/Cylinder.033.stl scale=1.000 1.000 0.833
- link Bottom_Link_1: mass 24.833333 -> 24.83
- link Bottom_Link_2: mass 24.833333 -> 24.83
- link Bottom_Link_3: mass 24.833333 -> 24.83
- link Colonna_Link_1: mass 8.60000 -> 8.6; geometry collision mesh filename=Robot/PIPPA/Cylinder.032.stl scale=0.060 0.060 0.100; visual mesh filename=Robot/PIPPA/Cylinder.032.stl scale=0.060 0.060 0.100
- link Colonna_Link_2: mass 8.60000 -> 8.6; geometry collision mesh filename=Robot/PIPPA/Cylinder.030.stl scale=0.060 0.060 0.100; visual mesh filename=Robot/PIPPA/Cylinder.030.stl scale=0.060 0.060 0.100
- link Colonna_Link_3: mass 8.60000 -> 8.6; geometry collision mesh filename=Robot/PIPPA/Cylinder.031.stl scale=0.060 0.060 0.100; visual mesh filename=Robot/PIPPA/Cylinder.031.stl scale=0.060 0.060 0.100
- link Cover_Link1: geometry collision mesh filename=Robot/PIPPA/Cylinder.029.stl scale=0.030 0.030 0.105; visual mesh filename=Robot/PIPPA/Cylinder.029.stl scale=0.030 0.030 0.105
- link Cover_Link_2: geometry collision mesh filename=Robot/PIPPA/Cylinder.027.stl scale=0.030 0.030 0.105; visual mesh filename=Robot/PIPPA/Cylinder.027.stl scale=0.030 0.030 0.105
- link Cover_Link_3: geometry collision mesh filename=Robot/PIPPA/Cylinder.028.stl scale=0.030 0.030 0.105; visual mesh filename=Robot/PIPPA/Cylinder.028.stl scale=0.030 0.030 0.105
- link Elastic_Joint_Link_1: geometry collision mesh filename=Robot/PIPPA/Cylinder.023.stl scale=0.006 0.005 0.040; visual mesh filename=Robot/PIPPA/Cylinder.023.stl scale=0.006 0.005 0.040
- link Elastic_Joint_link_2: geometry collision mesh filename=Robot/PIPPA/Cylinder.010.stl scale=0.006 0.005 0.040; visual mesh filename=Robot/PIPPA/Cylinder.010.stl scale=0.006 0.005 0.040
- link Elastic_Joint_link_3: geometry collision mesh filename=Robot/PIPPA/Cylinder.011.stl scale=0.006 0.005 0.040; visual mesh filename=Robot/PIPPA/Cylinder.011.stl scale=0.006 0.005 0.040
- link Gamba_Link_1: geometry collision mesh filename=Robot/PIPPA/Cylinder.026.stl scale=0.030 0.030 0.330; visual mesh filename=Robot/PIPPA/Cylinder.026.stl scale=0.030 0.030 0.330
- link Gamba_Link_2: geometry collision mesh filename=Robot/PIPPA/Cylinder.024.stl scale=0.030 0.030 0.330; visual mesh filename=Robot/PIPPA/Cylinder.024.stl scale=0.030 0.030 0.330
- link Gamba_Link_3: geometry collision mesh filename=Robot/PIPPA/Cylinder.025.stl scale=0.030 0.030 0.330; visual mesh filename=Robot/PIPPA/Cylinder.025.stl scale=0.030 0.030 0.330
- link Top_Link_1: geometry collision box size=0.040 0.340 0.030; visual mesh filename=Robot/PIPPA/Cube.006.stl scale=0.020 0.170 0.015
- link Top_Link_2: geometry collision box size=0.040 0.340 0.030; visual mesh filename=Robot/PIPPA/Cube.004.stl scale=0.020 0.170 0.015
- link Top_Link_3: geometry collision box size=0.040 0.340 0.030; visual mesh filename=Robot/PIPPA/Cube.005.stl scale=0.020 0.170 0.015
- link Top_core: mass 36.6000 -> 36.6; geometry collision mesh filename=Robot/PIPPA/Cylinder.003.stl scale=0.375 0.375 0.015; visual mesh filename=Robot/PIPPA/Cylinder.003.stl scale=0.375 0.375 0.015
Joints:
- removed joint Bottom_straight_to_1
- removed joint Bottom_straight_to__3
- removed joint Bottom_stright_to_2
- added joint Center_to_bottom1: type fixed, parent Colonna_Link_1, child Bottom_Link_1, origin xyz=-0.425 0.000 0.000 rpy=1.571 0.000 1.571
- added joint Center_to_bottom2: type fixed, parent Colonna_Link_2, child Bottom_Link_2, origin xyz=0.212 -0.368 0.000 rpy=1.571 -0.000 -2.618
- added joint Top_core_to__top_link: type fixed, parent Bottom_core, child Top_core, origin xyz=0.000 0.000 1.043 rpy=-3.142 0.000 0.000
- added joint center_to_bottom3: type fixed, parent Colonna_Link_3, child Bottom_Link_3, origin xyz=0.212 0.368 0.000 rpy=1.571 0.000 -0.524
- joint Bottom_to_Column_1: origin xyz=-0.00000 0.00000 -0.20000 rpy=0.00000 0.00000 0.00000 -> xyz=-0.000 0.000 -0.200 rpy=0.000 0.000 0.000
- joint Bottom_to_column3: origin xyz=0.00000 0.00000 -0.20000 rpy=0.00000 0.00000 0.00000 -> xyz=0.000 0.000 -0.200 rpy=0.000 0.000 0.000
- joint Bottom_to_column_2: origin xyz=0.00000 0.00000 -0.20000 rpy=0.00000 0.00000 0.00000 -> xyz=0.000 0.000 -0.200 rpy=0.000 0.000 0.000
- joint Cover_to_leg_1: origin xyz=0.10300 0.00000 0.42500 rpy=0.00000 -1.57080 0.00000 -> xyz=0.103 0.000 0.425 rpy=0.000 -1.571 0.000
- joint Cover_to_leg_2: origin xyz=0.10300 0.00028 0.42451 rpy=1.57080 0.52360 -1.57080 -> xyz=0.103 0.000 0.425 rpy=1.571 0.524 -1.571
- joint Cover_to_leg_3: origin xyz=0.10300 -0.00028 0.42451 rpy=-1.57080 0.52360 1.57080 -> xyz=0.103 -0.000 0.425 rpy=-1.571 0.524 1.571
- joint Cover_to_top_1: origin xyz=0.00000 0.00000 0.00000 rpy=-3.14159 -1.57080 0.00000 -> xyz=0.000 0.000 0.000 rpy=-3.142 -1.571 0.000
- joint Cover_to_top_2: origin xyz=0.00000 0.00000 0.00000 rpy=-0.35088 -1.57080 1.39808 -> xyz=0.000 0.000 0.000 rpy=-0.351 -1.571 1.398
- joint Cover_to_top_3: origin xyz=0.00000 0.00000 0.00000 rpy=-1.04720 -1.57080 0.00000 -> xyz=0.000 0.000 0.000 rpy=-1.047 -1.571 0.000
- joint Leg_to_elastic_1: origin xyz=0.00000 0.00000 -0.66000 rpy=0.00000 0.00000 0.00000 -> xyz=0.000 0.000 -0.660 rpy=0.000 0.000 0.000
- joint Leg_to_elastic_2: origin xyz=-0.00000 -0.00000 -0.66000 rpy=0.00000 0.00000 -0.00000 -> xyz=-0.000 0.000 -0.660 rpy=0.000 0.000 -0.000
- joint Leg_to_elastic_3: origin xyz=0.00000 0.00000 -0.66000 rpy=0.00000 0.00000 0.00000 -> xyz=0.000 0.000 -0.660 rpy=0.000 0.000 0.000
- joint elastic_to_column_1: origin xyz=0.00000 0.00000 -0.08000 rpy=0.00000 0.00000 0.00000 -> xyz=0.000 0.000 -0.080 rpy=0.000 0.000 0.000
- joint elastic_to_column_2: origin xyz=0.00000 -0.00000 -0.08000 rpy=0.00000 0.00000 0.00000 -> xyz=0.000 0.000 -0.080 rpy=0.000 0.000 0.000
- joint elastic_to_column_3: origin xyz=0.00000 0.00000 -0.08000 rpy=0.00000 0.00000 0.00000 -> xyz=0.000 0.000 -0.080 rpy=0.000 0.000 0.000

Commit message: Update PIPPA.urdf
Added mass to bottom core link

File: Robot/PIPPA/PIPPA.urdf (robot description, URDF)
Before this commit: robot PIPPA, 20 links, 19 joints
Links:
- link Bottom_Link_1: mass 24.83 -> 18.625
- link Bottom_Link_2: mass 24.83 -> 18.625
- link Bottom_Link_3: mass 24.83 -> 18.625
- link Bottom_core: mass 0 -> 18.625

Commit message: Update PIPPA.urdf

File: Robot/PIPPA/PIPPA.urdf (robot description, URDF)
Before this commit: robot PIPPA, 20 links, 19 joints
Links:
- link Bottom_Link_1: mass 18.625 -> 24
- link Bottom_Link_2: mass 18.625 -> 24
- link Bottom_Link_3: mass 18.625 -> 24
- link Bottom_core: mass 18.625 -> 2.5

Commit message: Update PIPPA.urdf

File: Robot/PIPPA/PIPPA.urdf (robot description, URDF)
Before this commit: robot PIPPA, 19 links, 18 joints
Links:
- link Top_Link_1: geometry collision box size=0.040 0.340 0.030; visual mesh filename=Robot/PIPPA/Cube.006.stl scale=0.020 0.170 0.015

Commit message: Update PIPPA.urdf

File: Robot/PIPPA/PIPPA.urdf (robot description, URDF)
Before this commit: robot PIPPA, 19 links, 18 joints
Links:
- link Bottom_Link_2: geometry collision mesh filename=Robot/PIPPA/Cylinder.033.stl scale=1.000 1.000 0.833; visual mesh filename=Robot/PIPPA/Cylinder.033.stl scale=1.000 1.000 0.833
- link Colonna_Link_1: geometry collision mesh filename=Robot/PIPPA/Cylinder.032.stl scale=0.060 0.060 0.100; visual mesh filename=Robot/PIPPA/Cylinder.032.stl scale=0.060 0.060 0.100

Commit message: Add files via upload

File: Robot/PIPPA/PIPPA.urdf (robot description, URDF)
Before this commit: robot PIPPA, 19 links, 18 joints
Links:
- removed link Cover_Link1
- removed link Top_core
- added link Cover_Link_1, mass 0.78; collision mesh filename=Robot/PIPPA/Cylinder.013.stl scale=0.030 0.030 0.105; visual mesh filename=Robot/PIPPA/Cylinder.013.stl scale=0.030 0.030 0.105
- added link Top_core_Link, mass 186.6; collision mesh filename=Robot/PIPPA/Cylinder.001.stl scale=0.375 0.375 0.015; visual mesh filename=Robot/PIPPA/Cylinder.001.stl scale=0.375 0.375 0.015
- link Bottom_Link_2: geometry collision mesh filename=Robot/PIPPA/Cylinder.017.stl scale=1.000 1.000 0.833; visual mesh filename=Robot/PIPPA/Cylinder.017.stl scale=1.000 1.000 0.833
- link Colonna_Link_1: geometry collision mesh filename=Robot/PIPPA/Cylinder.016.stl scale=0.060 0.060 0.100; visual mesh filename=Robot/PIPPA/Cylinder.016.stl scale=0.060 0.060 0.100
- link Colonna_Link_2: geometry collision mesh filename=Robot/PIPPA/Cylinder.014.stl scale=0.060 0.060 0.100; visual mesh filename=Robot/PIPPA/Cylinder.014.stl scale=0.060 0.060 0.100
- link Colonna_Link_3: geometry collision mesh filename=Robot/PIPPA/Cylinder.015.stl scale=0.060 0.060 0.100; visual mesh filename=Robot/PIPPA/Cylinder.015.stl scale=0.060 0.060 0.100
- link Cover_Link_2: geometry collision mesh filename=Robot/PIPPA/Cylinder.009.stl scale=0.030 0.030 0.105; visual mesh filename=Robot/PIPPA/Cylinder.009.stl scale=0.030 0.030 0.105
- link Cover_Link_3: geometry collision mesh filename=Robot/PIPPA/Cylinder.012.stl scale=0.030 0.030 0.105; visual mesh filename=Robot/PIPPA/Cylinder.012.stl scale=0.030 0.030 0.105
- link Elastic_Joint_Link_1: geometry collision mesh filename=Robot/PIPPA/Cylinder.005.stl scale=0.006 0.005 0.040; visual mesh filename=Robot/PIPPA/Cylinder.005.stl scale=0.006 0.005 0.040
- link Elastic_Joint_link_2: geometry collision mesh filename=Robot/PIPPA/Cylinder.002.stl scale=0.006 0.005 0.040; visual mesh filename=Robot/PIPPA/Cylinder.002.stl scale=0.006 0.005 0.040
- link Elastic_Joint_link_3: geometry collision mesh filename=Robot/PIPPA/Cylinder.004.stl scale=0.006 0.005 0.040; visual mesh filename=Robot/PIPPA/Cylinder.004.stl scale=0.006 0.005 0.040
- link Gamba_Link_1: geometry collision mesh filename=Robot/PIPPA/Cylinder.008.stl scale=0.030 0.030 0.330; visual mesh filename=Robot/PIPPA/Cylinder.008.stl scale=0.030 0.030 0.330
- link Gamba_Link_2: geometry collision mesh filename=Robot/PIPPA/Cylinder.006.stl scale=0.030 0.030 0.330; visual mesh filename=Robot/PIPPA/Cylinder.006.stl scale=0.030 0.030 0.330
- link Gamba_Link_3: geometry collision mesh filename=Robot/PIPPA/Cylinder.007.stl scale=0.030 0.030 0.330; visual mesh filename=Robot/PIPPA/Cylinder.007.stl scale=0.030 0.030 0.330
- link Top_Link_1: geometry collision mesh filename=Robot/PIPPA/Cube.009.stl scale=0.020 0.170 0.015; visual mesh filename=Robot/PIPPA/Cube.009.stl scale=0.020 0.170 0.015
- link Top_Link_2: geometry collision mesh filename=Robot/PIPPA/Cube.007.stl scale=0.020 0.170 0.015; visual mesh filename=Robot/PIPPA/Cube.007.stl scale=0.020 0.170 0.015
- link Top_Link_3: geometry collision mesh filename=Robot/PIPPA/Cube.008.stl scale=0.020 0.170 0.015; visual mesh filename=Robot/PIPPA/Cube.008.stl scale=0.020 0.170 0.015
Joints:
- joint Center_to_bottom2: origin xyz=0.212 -0.368 0.000 rpy=1.571 -0.000 -2.618 -> xyz=0.212 -0.368 0.000 rpy=1.571 0.000 -2.618
- joint Cover_to_leg_1: child Cover_Link1 -> Cover_Link_1
- joint Cover_to_top_1: parent Top_core -> Top_core_Link
- joint Cover_to_top_2: parent Top_core -> Top_core_Link
- joint Cover_to_top_3: parent Top_core -> Top_core_Link
- joint Leg_to_elastic_1: parent Cover_Link1 -> Cover_Link_1
- joint center_to_bottom3: origin xyz=0.212 0.368 0.000 rpy=1.571 0.000 -0.524 -> xyz=0.212 0.368 0.000 rpy=2.094 1.571 0.000
