Commit message: Update PIPPA_oneleg.urdf

File: Robot/1LegTrail/PIPPA_oneleg.urdf (robot description, URDF)
Before this commit: robot PIPPA_oneleg, 3 links, 2 joints
Links:
- link Gamba_Link: geometry collision cylinder length=0.675 radius=0.03; visual cylinder length=0.675 radius=0.03
- link Giunto_Link: mass None -> 0.0569; geometry collision cylinder length=0.08 radius=0.0055; visual cylinder length=0.08 radius=0.0055
- link Link_colonna: geometry collision cylinder length=0.2 radius=0.06; visual cylinder length=0.2 radius=0.06
Joints:
- removed joint Gamba_Link_joint
- removed joint Giunto_Link_joint
- added joint Colonna_Giunto_joint: type fixed, parent Link_colonna, child Giunto_Link, origin xyz=0 0 0.2 rpy=0 0 0
- added joint Giunto_Gamba_joint: type fixed, parent Giunto_Link, child Gamba_Link, origin xyz=0 0 0.08 rpy=0 0 0

Commit message: Added soft body

File: Robot/1LegTrail/PIPPA_oneleg.urdf (robot description, URDF)
Before this commit: robot PIPPA_oneleg, 3 links, 2 joints
Links:
- link Giunto_Link: mass 0.0569 -> None

Commit message: Update PIPPA_oneleg.urdf

File: Robot/1LegTrail/PIPPA_oneleg.urdf (robot description, URDF)
Before this commit: robot PIPPA_oneleg, 3 links, 2 joints
Joints:
- joint Giunto_Gamba_joint: axis (none) -> 0 1 0; type fixed -> revolute

Commit message: Update PIPPA_oneleg.urdf

File: Robot/1LegTrail/PIPPA_oneleg.urdf (robot description, URDF)
Before this commit: robot PIPPA_oneleg, 3 links, 2 joints
Joints:
- joint Giunto_Gamba_joint: axis 0 1 0 -> (none); type revolute -> fixed

Commit message: Update PIPPA_oneleg.urdf

File: Robot/1LegTrail/PIPPA_oneleg.urdf (robot description, URDF)
Before this commit: robot PIPPA_oneleg, 3 links, 2 joints
Links:
- link Giunto_Link: mass None -> 0.0569
